File: Board/PowerSenseModule/sensing.sch (KiCad schematic (older format))
At the start: 21 parts, among them U5 MCP9700AT-ETT, U6 MCP39F511A

Commit message: PCB Design Began. Design Changes are incoming though.
PCB placement began, changes to schematic will be made. Reference google docs for said changes along with date.
Parts:
- C16, C17: value 3.0nF -> 3.3nF
- C19, C22: footprint Capacitor_SMD:C_0603_1608Metric_Pad1.05x0.95mm_HandSolder -> Capacitor_SMD:C_0805_2012Metric_Pad1.15x1.40mm_HandSolder
Changed lines of the file:
@@
 F 0 "C19" H 5215 1996 50  0000 L CNN
 F 1 "1uF" H 5215 1905 50  0000 L CNN
-F 2 "Capacitor_SMD:C_0603_1608Metric_Pad1.05x0.95mm_HandSolder" H 5138 1800 50  0001 C CNN
+F 2 "Capacitor_SMD:C_0805_2012Metric_Pad1.15x1.40mm_HandSolder" H 5138 1800 50  0001 C CNN
 F 3 "~" H 5100 1950 50  0001 C CNN
 	1    5100 1950
@@
 F 0 "C22" H 7665 4246 50  0000 L CNN
 F 1 "1uF" H 7665 4155 50  0000 L CNN
-F 2 "Capacitor_SMD:C_0603_1608Metric_Pad1.05x0.95mm_HandSolder" H 7588 4050 50  0001 C CNN
+F 2 "Capacitor_SMD:C_0805_2012Metric_Pad1.15x1.40mm_HandSolder" H 7588 4050 50  0001 C CNN
 F 3 "~" H 7550 4200 50  0001 C CNN
 	1    7550 4200
@@
 P 3300 2750
 F 0 "C16" H 3415 2796 50  0000 L CNN
-F 1 "3.0nF" H 3415 2705 50  0000 L CNN
+F 1 "3.3nF" H 3415 2705 50  0000 L CNN
 F 2 "Capacitor_SMD:C_0603_1608Metric_Pad1.05x0.95mm_HandSolder" H 3338 2600 50  0001 C CNN
 F 3 "~" H 3300 2750 50  0001 C CNN
@@
 P 3800 2750
 F 0 "C17" H 3915 2796 50  0000 L CNN
-F 1 "3.0nF" H 3915 2705 50  0000 L CNN
+F 1 "3.3nF" H 3915 2705 50  0000 L CNN
 F 2 "Capacitor_SMD:C_0603_1608Metric_Pad1.05x0.95mm_HandSolder" H 3838 2600 50  0001 C CNN
 F 3 "~" H 3800 2750 50  0001 C CNN
