File: Board/PowerSenseModule/sensing.sch (KiCad schematic (older format))
At the start: 21 parts, among them U5 MCP9700AT-ETT, U6 MCP39F511A

Commit message: Started design change
Changing MCU to 5V dspic33ev32gm102
Parts:
- removed C16, C17: 3.3nF, Capacitor_SMD:C_0603_1608Metric_Pad1.05x0.95mm_HandSolder, symbol Device:C
- removed C18: 820pF, Capacitor_SMD:C_0603_1608Metric_Pad1.05x0.95mm_HandSolder, symbol Device:C
- removed C19, C22: 1uF, Capacitor_SMD:C_0805_2012Metric_Pad1.15x1.40mm_HandSolder, symbol Device:C
- removed C20, C23, C24: 0.1uF, Capacitor_SMD:C_0603_1608Metric_Pad1.05x0.95mm_HandSolder, symbol Device:C
- removed C21: 0.01uF, Capacitor_SMD:C_0603_1608Metric_Pad1.05x0.95mm_HandSolder, symbol Device:C
- removed R10, R11, R14: 1k, Resistor_SMD:R_0603_1608Metric_Pad1.05x0.95mm_HandSolder, symbol Device:R_US
- removed R12, R9: 499k, Resistor_SMD:R_0603_1608Metric_Pad1.05x0.95mm_HandSolder, symbol Device:R_US
- removed R13: 34.8k, Resistor_SMD:R_0603_1608Metric_Pad1.05x0.95mm_HandSolder, symbol Device:R_US
- removed R15, R17: 10k, Resistor_SMD:R_0603_1608Metric_Pad1.05x0.95mm_HandSolder, symbol Device:R_US
- removed R16: 10, Resistor_SMD:R_0603_1608Metric_Pad1.05x0.95mm_HandSolder, symbol Device:R_US
- removed U5: MCP9700AT-ETT, Package_TO_SOT_SMD:SOT-23, symbol Sensor_Temperature:MCP9700AT-ETT
- removed U6: MCP39F511A, Package_DFN_QFN:QFN-28-1EP_5x5mm_P0.5mm_EP3.35x3.35mm, symbol F1_Power_Sense:MCP39F511A
Connections:
- net labels removed: +3V3, GNDA, GNDD, PSEN_ADC_RST, PSEN_EVENT1, PSEN_EVENT2, PSEN_MCLR, PSEN_UART_RX, PSEN_UART_TX, PSEN_ZCD
- wire segments 63 -> 2
Other:
- note removed: "The exposed pad should be connected to GNDD\n"
- note removed: "Using internal oscillator\n"
