File: Board/PowerSenseModule/_autosave-PowerSenseModule.kicad_pcb (KiCad board)
At the start: 2 copper layers, 114.3 x 55.9 mm, 54 parts, among them J1 Conn_01x06_Male, J3 Programming Header, J4 Conn_01x02_Male, U1 TPS82150, U2 NCV2007x, U3 dsPIC33EV32GM102, U4 MCP2542FDxMF, Y1 Crystal

Commit message: misc - PCB
Parts:
- moved R7 103.6 mm to (208.3, 46.1)
- moved U4 103.6 mm to (208.3, 42.3)
- moved R12 43.9 mm to (212.0, 98.3)
- moved C18 37.5 mm to (184.8, 68.7), turned to 270 degrees
- moved C15 36.8 mm to (182.9, 74.0), turned to 90 degrees
- moved D3 36.1 mm to (182.1, 85.0), turned to 90 degrees
- moved R20 36.0 mm to (182.1, 81.2), turned to 90 degrees
- moved R18 35.6 mm to (211.8, 100.7), turned to 0 degrees
- moved R19 34.7 mm to (212.0, 95.5), turned to 180 degrees
- moved Y1 34.4 mm to (187.5, 68.7), turned to 270 degrees
- moved D4 33.2 mm to (184.2, 85.0), turned to 90 degrees
- moved R21 32.9 mm to (184.3, 81.2), turned to 90 degrees
- moved C7 32.5 mm to (170.6, 80.4)
- moved C8 32.5 mm to (175.3, 72.4)
- moved R1 32.5 mm to (170.6, 78.4)
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Routing:
- net Net-(R11-Pad1): track 6.85 -> 0.00 mm
- net Net-(R10-Pad1): track 4.45 -> 0.00 mm
- net Net-(R11-Pad2): track 3.38 -> 0.24 mm
- net Net-(R13-Pad1): track 2.76 -> 0.00 mm
Other:
- net class Default: trace_width 0.25 -> 48.9
- rule trace_min: 0.2 -> 48.7
