File: Board/PowerSenseModule/PowerSenseModule.sch (KiCad schematic (older format))
At the start: 24 parts, among them J1 Conn_01x06_Male, U1 TPS82150

Commit message: Added info in symbol fields for diodes
Parts:
- D2, D5, D6, D7: Manufacturer (none) -> Toshiba; Manufacturer PN (none) -> CUS10S30,H3F; Price 1 QTY (none) -> 0.42; Supplier (none) -> Mouser; Supplier PN (none) -> 757-CUS10S30H3F
Changed lines of the file:
@@
 F 3 "http://toshiba.semicon-storage.com/ap-en/product/diode/sbd/detail.CUS10S30.html" H 7300 4175 50  0001 C CNN
 F 4 "https://www.mouser.com/ProductDetail/Toshiba/CUS10S30H3F?qs=sGAEpiMZZMtQ8nqTKtFS%2FLnbHK8U7YHpoD%2FnZkbvIUu50yFANYtBSg%3D%3D" H 7300 4175 50  0001 C CNN "Supplier Link"
+F 5 "Toshiba" H 7300 4175 50  0001 C CNN "Manufacturer"
+F 6 "CUS10S30,H3F" H 7300 4175 50  0001 C CNN "Manufacturer PN"
+F 7 "0.42" H 7300 4175 50  0001 C CNN "Price 1 QTY"
+F 8 "Mouser" H 7300 4175 50  0001 C CNN "Supplier"
+F 9 " 757-CUS10S30H3F " H 7300 4175 50  0001 C CNN "Supplier PN"
 	1    7300 4175
 	-1   0    0    1
@@
 F 3 "http://toshiba.semicon-storage.com/ap-en/product/diode/sbd/detail.CUS10S30.html" H 7825 4175 50  0001 C CNN
 F 4 "https://www.mouser.com/ProductDetail/Toshiba/CUS10S30H3F?qs=sGAEpiMZZMtQ8nqTKtFS%2FLnbHK8U7YHpoD%2FnZkbvIUu50yFANYtBSg%3D%3D" H 7825 4175 50  0001 C CNN "Supplier Link"
+F 5 "Toshiba" H 7825 4175 50  0001 C CNN "Manufacturer"
+F 6 "CUS10S30,H3F" H 7825 4175 50  0001 C CNN "Manufacturer PN"
+F 7 "0.42" H 7825 4175 50  0001 C CNN "Price 1 QTY"
+F 8 "Mouser" H 7825 4175 50  0001 C CNN "Supplier"
+F 9 " 757-CUS10S30H3F " H 7825 4175 50  0001 C CNN "Supplier PN"
 	1    7825 4175
 	-1   0    0    1
@@
 F 3 "http://toshiba.semicon-storage.com/ap-en/product/diode/sbd/detail.CUS10S30.html" H 8450 4175 50  0001 C CNN
 F 4 "https://www.mouser.com/ProductDetail/Toshiba/CUS10S30H3F?qs=sGAEpiMZZMtQ8nqTKtFS%2FLnbHK8U7YHpoD%2FnZkbvIUu50yFANYtBSg%3D%3D" H 8450 4175 50  0001 C CNN "Supplier Link"
+F 5 "Toshiba" H 8450 4175 50  0001 C CNN "Manufacturer"
+F 6 "CUS10S30,H3F" H 8450 4175 50  0001 C CNN "Manufacturer PN"
+F 7 "0.42" H 8450 4175 50  0001 C CNN "Price 1 QTY"
+F 8 "Mouser" H 8450 4175 50  0001 C CNN "Supplier"
+F 9 " 757-CUS10S30H3F " H 8450 4175 50  0001 C CNN "Supplier PN"
 	1    8450 4175
 	-1   0    0    1
@@
 F 3 "http://toshiba.semicon-storage.com/ap-en/product/diode/sbd/detail.CUS10S30.html" H 8975 4175 50  0001 C CNN
 F 4 "https://www.mouser.com/ProductDetail/Toshiba/CUS10S30H3F?qs=sGAEpiMZZMtQ8nqTKtFS%2FLnbHK8U7YHpoD%2FnZkbvIUu50yFANYtBSg%3D%3D" H 8975 4175 50  0001 C CNN "Supplier Link"
+F 5 "Toshiba" H 8975 4175 50  0001 C CNN "Manufacturer"
+F 6 "CUS10S30,H3F" H 8975 4175 50  0001 C CNN "Manufacturer PN"
+F 7 "0.42" H 8975 4175 50  0001 C CNN "Price 1 QTY"
+F 8 "Mouser" H 8975 4175 50  0001 C CNN "Supplier"
+F 9 " 757-CUS10S30H3F " H 8975 4175 50  0001 C CNN "Supplier PN"
 	1    8975 4175
 	-1   0    0    1
