File: Board/PowerSenseModule/PowerSenseModule_alt.kicad_pcb (KiCad board)
At the start: 2 copper layers, 91.1 x 62.3 mm, 71 parts, among them J1 DT13-6P, J3 Programming Header, J4 Board Interconnect, U1 TPS82150, U2 NCV2007x, U3 dsPIC33EV32GM102, U4 MCP2542FDxMF, Y1 25 MHz

Commit message: Added drawings dimensions, changed footprint of op amp, and cleaned up
Parts:
- J1: value DT13-6P -> CONN6_DT13-6P
- moved C23 1.71 mm to (159.7, 79.8)
- moved J4 0.15 mm to (152.3, 90.5)
- moved U2 0.07 mm to (160.9, 91.9)
Routing:
- net GNDA: track 25.2 -> 29.5 mm
- net Net-(R18-Pad1): track 8.42 -> 10.2 mm
- net /PWM: track 42.7 -> 41.1 mm
- net Net-(R11-Pad2): track 5.50 -> 6.77 mm
- net /MCU and CAN/VSENSE: track 11.4 -> 10.4 mm
- net /MCU and CAN/SENSE+: track 19.9 -> 19.2 mm
- net Net-(R10-Pad1): track 33.3 -> 34.0 mm
- net /MCU and CAN/SENSE-: track 19.8 -> 20.4 mm
- net Net-(R22-Pad2): track 9.37 -> 9.88 mm
- net GND: vias 88 -> 70
- net (no net): vias 1 -> 0
